File: DevBuddy_mk1/DevBuddy/ADC_Channels.kicad_sch (KiCad schematic)
At the start: 12 parts, among them U2 74HC4051, U3 74HC4051, U4 INA190A2IDCKR

Commit message: Heavy additions to schematic
Parts:
- removed R4: 15mR, Resistor_SMD:R_2512_6332Metric, symbol Device:R_Small
- added C120: 100n, Capacitor_SMD:C_0402_1005Metric, symbol Device:C_Small
- added R60: 10R, Resistor_SMD:R_0402_1005Metric, symbol Device:R_Small
- added R62: 8k6, Resistor_SMD:R_0402_1005Metric, symbol Device:R_Small
- added R63, R65, R67, R69, R71, R73, R75: 100k, Resistor_SMD:R_0402_1005Metric, symbol Device:R_Small
- added R64, R70: 28k, Resistor_SMD:R_0402_1005Metric, symbol Device:R_Small
- added R66: 200k, Resistor_SMD:R_0402_1005Metric, symbol Device:R_Small
- added R68, R72, R74, R76: 56k, Resistor_SMD:R_0402_1005Metric, symbol Device:R_Small
- added U16: 74HC4051, Package_SO:SOIC-16_3.9x9.9mm_P1.27mm, symbol 74xx:74HC4051
- R2: value 100R -> 10R; footprint Resistor_SMD:R_01005_0402Metric -> Resistor_SMD:R_0402_1005Metric
- R3: value 100R -> 100k; footprint Resistor_SMD:R_01005_0402Metric -> Resistor_SMD:R_0402_1005Metric
Connections:
- net +3V3: now also C120.1, U16.16 (VCC)
- net ADC_in_Hi: now also R60.1; no longer R2.1
- net ADC_in_Low: now also R2.1, U16.3 (A); no longer R3.2
- net GND: now also C120.2, R62.1, R64.1, R66.1, R68.1, R70.1, R72.1, R74.1, R76.1, U16.6 (~{E}), U16.7 (VEE), U16.8 (GND)
- net MUX_S0: now also U16.11 (S0)
- net MUX_S1: now also U16.10 (S1)
- net MUX_S2: now also U16.9 (S2)
- net at C5.1, C8.1, U4.4 (IN+): now also R60.2; no longer R2.2
- net at C5.2, C7.1, U4.5 (IN-): now also R2.2; no longer R3.1
- net ADC_R2_Hi renamed 12V_C_CurSense_Hi
- net ADC_R2_Low renamed 12V_C_CurSense_Low
- net ADC_R3_Hi renamed 3V3_C_CurSense_Hi
- net ADC_R3_Low renamed 3V3_C_CurSense_Low
- net ADC_R4_Hi renamed 5V_C_CurSense_Hi
- net ADC_R4_Low renamed 5V_C_CurSense_Low
- net ADC_R5_Hi renamed 12V_D_CurSense_Hi
- net ADC_R5_Low renamed 12V_D_CurSense_Low
- net ADC_R6_Hi renamed 5V_D_CurSense_Hi
- net ADC_R6_Low renamed 5V_D_CurSense_Low
- net ADC_R7_Hi renamed Var_V2_CurSense_Hi
- net ADC_R7_Low renamed Var_V2_CurSense_Low
- net ADC_R8_Hi renamed Var_V1_CurSense_Hi
- net ADC_R8_Low renamed Var_V1_CurSense_Low
- net ADC_out_v renamed ACV_Curr_Out
- new net +12VDC_C: R63.2
- new net +12VDC_D: R69.2
- new net +3V3_C: R65.2
- new net +5V_C: R67.2
- new net +5V_D: R71.2
- new net +Var_V_1: R73.2
- new net +Var_V_2: R75.2
- new net VCC: R3.2
- new net V_Meas_0: R3.1, R62.2, U16.13 (A0)
- new net V_Meas_1: R63.1, R64.2, U16.14 (A1)
- new net V_Meas_2: R65.1, R66.2, U16.15 (A2)
- new net V_Meas_3: R67.1, R68.2, U16.12 (A3)
- new net V_Meas_4: R69.1, R70.2, U16.1 (A4)
- new net V_Meas_5: R71.1, R72.2, U16.5 (A5)
- new net V_Meas_6: R73.1, R74.2, U16.2 (A6)
- new net V_Meas_7: R75.1, R76.2, U16.4 (A7)
Other:
- note added: "+12VDC_C: Up to 12V Divider gives 3.28V for 15V in"
- note added: "+12VDC_D: Up to 12V Divider gives 3.28V for 15V in"
- note added: "+3V3_C: Up to 3.3V Divider gives 3.33V for 5V in"
- note added: "+5V_C: Up to 5V Divider gives 3.23V for 9V in"
- note added: "+5V_D: Up to 5V Divider gives 3.23V for 9V in"
- note added: "12VDC_C"
- note added: "12V_D"
- note added: "3V3_C"
- note added: "5V_C"
- note added: "5V_D"
- note added: "ADC Current MUX AND INA"
- note added: "ADC Voltage Mux"
- note added: "Current differential voltages"
- note added: "Safe voltage channels for MUX"
- note added: "VCC: Up to 28V Divider gives 3.16V for 40V in"
- note added: "Var_V1"
- note added: "Var_V2"
- note added: "Vin"
- note removed: "ADC MUX AND INA"

Commit message: More work into the PCB, mainly connectors
Connections:
- net ADC_in_Low: no longer U16.3 (A)
- new net ACV_Vol_Out: U16.3 (A)
Changed lines of the file:
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@@
+	(wire
+		(pts
+			(xy 166.37 53.34) (xy 168.91 53.34)
+		)
+		(stroke
+			(width 0)
+			(type default)
+		)
+	)
 	(wire
 		(pts
@@
 		(pts
 			(xy 361.95 76.2) (xy 361.95 78.74)
-		)
-		(stroke
-			(width 0)
-			(type default)
-		)
-	)
-	(wire
-		(pts
-			(xy 157.48 53.34) (xy 168.91 53.34)
 		)
 		(stroke
@@
 		)
 	)
-	(label "ADC_in_Low"
-		(at 157.48 53.34 0)
-		(effects
-			(font
-				(size 1.27 1.27)
-			)
-			(justify left bottom)
-		)
-	)
 	(label "ADC_R4_Hi"
 		(at 50.8 57.15 0)
@@
 		)
 	)
+	(global_label "ACV_Vol_Out"
+		(shape input)
+		(at 166.37 53.34 180)
+		(fields_autoplaced yes)
+		(effects
+			(font
+				(size 1.27 1.27)
+			)
+			(justify right)
+		)
+		(property "Intersheetrefs" "${INTERSHEET_REFS}"
+			(at 151.8944 53.34 0)
+			(effects
+				(font
+					(size 1.27 1.27)
+				)
+				(justify right)
+				(hide yes)
+			)
+		)
+	)

Commit message: PCB, starting the board
Connections:
- net ADC_R1_Hi renamed VCC_CurSense_Hi
- net ADC_R1_Low renamed VCC_CurSense_Low
Changed lines of the file:
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@@
+	(wire
+		(pts
+			(xy 62.23 160.02) (xy 68.58 160.02)
+		)
+		(stroke
+			(width 0)
+			(type default)
+		)
+	)
 	(wire
 		(pts
@@
 		(pts
 			(xy 38.1 104.14) (xy 40.64 104.14)
+		)
+		(stroke
+			(width 0)
+			(type default)
+		)
+	)
+	(wire
+		(pts
+			(xy 62.23 156.21) (xy 68.58 156.21)
 		)
 		(stroke
@@
 	)
 	(label "ADC_R1_Hi"
-		(at 68.58 161.29 0)
+		(at 68.58 160.02 0)
 		(effects
 			(font
@@
 	)
 	(label "ADC_R1_Low"
-		(at 68.58 157.48 0)
+		(at 68.58 156.21 0)
 		(effects
 			(font
@@
 			)
 			(justify left bottom)
+		)
+	)
+	(global_label "VCC_CurSense_Hi"
+		(shape input)
+		(at 62.23 160.02 180)
+		(fields_autoplaced yes)
+		(effects
+			(font
+				(size 1.27 1.27)
+			)
+			(justify right)
+		)
+		(property "Intersheetrefs" "${INTERSHEET_REFS}"
+			(at 42.9767 160.02 0)
+			(effects
+				(font
+					(size 1.27 1.27)
+				)
+				(justify right)
+				(hide yes)
+			)
 		)
 	)
@@
 			(effects
 				(font
+					(size 1.27 1.27)
+				)
+				(justify right)
+				(hide yes)
+			)
+		)
+	)
+	(global_label "VCC_CurSense_Low"
+		(shape input)
+		(at 62.23 156.21 180)
+		(fields_autoplaced yes)
+		(effects
+			(font
+				(size 1.27 1.27)
+			)
+			(justify right)
+		)
+		(property "Intersheetrefs" "${INTERSHEET_REFS}"
+			(at 41.4044 156.21 0)
+			(effects
+				(font
