File: DevBuddy_mk1/DevBuddy/Connectors.kicad_sch (KiCad schematic)
At the start: 43 parts, among them J2 Conn_01x02_Socket, J4 UART_Conns, J5 PC30, Q1 AO3415A, Q10 AO3415A, Q2 BC817, Q3 BC817, Q4 AO3415A, Q5 BC817, Q6 AO3415A, Q7 BC817, Q8 AO3415A, Q9 BC817, U17 TPS22965NQWDSGRQ1, U18 TPS22965NQWDSGRQ1, U19 TPS22965NQWDSGRQ1

Commit message: PCB, starting the board
Parts:
- added J6: Conn_01x15_Pin, Connector_PinHeader_2.54mm:PinHeader_1x15_P2.54mm_Vertical_SMD_Pin1Left, symbol Connector:Conn_01x15_Pin
- added R98: 20mOhm, Resistor_SMD:R_1210_3225Metric, symbol Device:R
Connections:
- net GND: now also J6.1 (Pin_1), J6.10 (Pin_10), J6.11 (Pin_11), J6.12 (Pin_12), J6.13 (Pin_13), J6.14 (Pin_14), J6.15 (Pin_15), J6.2 (Pin_2), J6.3 (Pin_3), J6.4 (Pin_4), J6.5 (Pin_5), J6.6 (Pin_6), J6.7 (Pin_7), J6.8 (Pin_8), J6.9 (Pin_9)
- net VCC: now also R98.2; no longer J2.2 (Pin_2)
- new net VCC_CurSense_Hi: J2.2 (Pin_2), R98.1
Other:
- note added: "PC30-PC15 Main Connectors"
- note removed: "PC30 Main Connector"
- moved on the sheet: J2
